Commit message: fix(gaden): elevate gas sensor to detect rising H2 gas
GADEN correctly simulates hydrogen gas rising to ceiling level
(~1.8m), but the sensor was positioned at only 0.45m height.

Changes:
- URDF: Raise gas_sensor_link from 0.45m to 1.5m
- scene.yaml: Use gas_sensor_link instead of base_link as sensor_frame
- test: Update assertions to match new configuration

Root cause analysis:
- H2 is 14x lighter than air, causing rapid vertical rise
- Filaments detected at 1.8-1.9m height in GADEN simulation
- Sensor at 0.45m could not detect rising gas plume
- After fix: Gas concentration readings 22-92 ppm (vs 0 before)

Co-Authored-By: Claude Opus 4.6 <noreply@anthropic.com>

File: src/h2track_sim/urdf/h2track_bot.urdf.xacro (robot description, xacro)
@@ -127,5 +127,6 @@
     <parent link="base_link"/>
     <child link="gas_sensor_link"/>
-    <origin xyz="0 0 0.45"/>
+    <!-- Elevated sensor height (1.5m) to detect rising H2 gas -->
+    <origin xyz="0 0 1.5"/>
   </joint>
   <gazebo reference="base_link">
